File: STM-LORA.sch (KiCad schematic (older format))
At the start: 2 parts, among them U1 stm32f103c8t6-module-china, U2 RFM95HW

Commit message: Added power components
Parts:
- added C1: 100µ, Discret:CP4, symbol CP
- added C2: 100n, Capacitors_ThroughHole:C_Disc_D6_P5, symbol C
- added D1: D_Schottky BAT85, Diodes_ThroughHole:Diode_DO-41_SOD81_Vertical_AnodeUp, symbol D_Schottky
- added R1, R2: 100k, Resistors_ThroughHole:Resistor_Vertical_RM5mm, symbol R
Connections:
- net labels added: +3.3V, +5V, +BATT, BattTest
- wire segments 26 -> 34
- no-connect marks 0 -> 31
Other:
- note added: "2.4V (2x AA(A) NiMH) or\n3.6V (3x AA(A) NiMH) or ..."
- note added: "Solar Panel (4V - ..)"

Commit message: update STM32 lib, add connectors
Parts:
- added J1: Batt, Pin_Headers:Pin_Header_Straight_1x02_Pitch2.54mm, symbol CONN_01X02_MALE
- added J2: Solar, Pin_Headers:Pin_Header_Straight_1x02_Pitch2.54mm, symbol CONN_01X02_MALE
- added J3: CONN_01X17, Socket_Strips:Socket_Strip_Straight_1x17_Pitch2.54mm, symbol CONN_01X17
- added J4, J5: CONN_01X03, Pin_Headers:Pin_Header_Straight_1x03_Pitch2.54mm, symbol CONN_01X03
- C1: footprint Discret:CP4 -> Capacitors_THT:CP_Radial_D6.3mm_P2.50mm
- C2: footprint Capacitors_ThroughHole:C_Disc_D6_P5 -> Capacitors_THT:C_Disc_D5.0mm_W2.5mm_P5.00mm
- D1: value D_Schottky BAT85 -> BAT85; footprint Diodes_ThroughHole:Diode_DO-41_SOD81_Vertical_AnodeUp -> Diodes_THT:D_DO-35_SOD27_P2.54mm_Vertical_AnodeUp
- R1, R2: footprint Resistors_ThroughHole:Resistor_Vertical_RM5mm -> Resistors_THT:R_Axial_DIN0309_L9.0mm_D3.2mm_P2.54mm_Vertical
Connections:
- net labels removed: +5V, +BATT
- wire segments 34 -> 83
- no-connect marks 31 -> 15

Commit message: start traces
Parts:
- added J6: CONN_01X01, symbol CONN_01X01
- added J7: CONN_01X14, symbol CONN_01X14
Connections:
- net labels added: P22, P25, P26, P27, P28, P29, P30, P31, P32, P33, P34, P35, P36, P37
- net labels removed: +3.3V, BattTest
- wire segments 83 -> 82
- no-connect marks 15 -> 7
Changed lines of the file:
@@
 	1    0    0    -1
 $EndComp
-Text Label 8450 3800 0    60   ~ 0
-BattTest
-Text Label 3950 4350 0    60   ~ 0
-BattTest
 $Comp
 L CP C1
@@
 	0    -1   -1   0
 $EndComp
-NoConn ~ 3900 2700
-NoConn ~ 3900 2850
-NoConn ~ 3900 3000
-NoConn ~ 3900 3900
-NoConn ~ 3900 4200
-NoConn ~ 3900 4500
-NoConn ~ 3900 4650
 NoConn ~ 3900 4800
-NoConn ~ 3900 4950
-NoConn ~ 3900 5100
 NoConn ~ 4700 3150
 NoConn ~ 5800 3500
@@
 	5800 3400 6000 3400
 Wire Wire Line
-	6000 3400 6000 5750
-Wire Wire Line
-	1100 5750 6000 5750
-Wire Wire Line
-	1100 2050 1100 5750
+	6000 3400 6000 6500
+Wire Wire Line
+	6000 6500 1100 6500
+Wire Wire Line
+	1100 6500 1100 2050
 Wire Wire Line
 	1100 4050 1800 4050
@@
 	8400 3800 8900 3800
 Connection ~ 8900 3800
-Wire Wire Line
-	3900 4350 4250 4350
 Connection ~ 8800 1900
 Wire Wire Line
@@
 	4700 3750 3900 3750
 Connection ~ 5000 2550
-$Comp
-L +3.3V #PWR015
-U 1 1 58DF97C4
-P 5000 2550
-F 0 "#PWR015" H 5000 2400 50  0001 C CNN
-F 1 "+3.3V" H 5000 2690 50  0000 C CNN
-F 2 "" H 5000 2550 50  0000 C CNN
-F 3 "" H 5000 2550 50  0000 C CNN
-	1    5000 2550
-	1    0    0    -1
-$EndComp
 Connection ~ 4400 2550
 Connection ~ 4800 2550
@@
 	4800 2100 4800 2550
 $Comp
-L GND #PWR016
+L GND #PWR015
 U 1 1 58DF9B90
 P 4800 1800
-F 0 "#PWR016" H 4800 1550 50  0001 C CNN
+F 0 "#PWR015" H 4800 1550 50  0001 C CNN
 F 1 "GND" H 4800 1650 50  0000 C CNN
 F 2 "" H 4800 1800 50  0000 C CNN
@@
 $EndComp
 $Comp
-L GND #PWR017
+L GND #PWR016
 U 1 1 58DF9BB7
 P 4400 1800
-F 0 "#PWR017" H 4400 1550 50  0001 C CNN
+F 0 "#PWR016" H 4400 1550 50  0001 C CNN
 F 1 "GND" H 4400 1650 50  0000 C CNN
 F 2 "" H 4400 1800 50  0000 C CNN
 F 3 "" H 4400 1800 50  0000 C CNN
 	1    4400 1800
-	-1   0    0    1
-$EndComp
-$Comp
-L PWR_FLAG #FLG018
-U 1 1 58DF9D30
-P 5000 2550
-F 0 "#FLG018" H 5000 2645 50  0001 C CNN
-F 1 "PWR_FLAG" H 5000 2730 50  0000 C CNN
-F 2 "" H 5000 2550 50  0000 C CNN
-F 3 "" H 5000 2550 50  0000 C CNN
-	1    5000 2550
 	-1   0    0    1
 $EndComp
@@
 $EndComp
 $Comp
-L GND #PWR019
+L GND #PWR017
 U 1 1 58DFA43D
 P 9100 2100
-F 0 "#PWR019" H 9100 1850 50  0001 C CNN
+F 0 "#PWR017" H 9100 1850 50  0001 C CNN
 F 1 "GND" H 9100 1950 50  0000 C CNN
 F 2 "" H 9100 2100 50  0001 C CNN
@@
 $EndComp
 $Comp
-L GND #PWR020
+L GND #PWR018
 U 1 1 58DFA51A
 P 9100 3050
-F 0 "#PWR020" H 9100 2800 50  0001 C CNN
+F 0 "#PWR018" H 9100 2800 50  0001 C CNN
 F 1 "GND" H 9100 2900 50  0000 C CNN
 F 2 "" H 9100 3050 50  0001 C CNN
@@
 	850  5100 1800 5100
 $Comp
-L GND #PWR021
+L GND #PWR019
 U 1 1 58E02B12
 P 850 5000
-F 0 "#PWR021" H 850 4750 50  0001 C CNN
+F 0 "#PWR019" H 850 4750 50  0001 C CNN
 F 1 "GND" H 850 4850 50  0000 C CNN
 F 2 "" H 850 5000 50  0001 C CNN
@@
 $EndComp
 $Comp
-L VCC #PWR022
+L VCC #PWR020
 U 1 1 58E02B47
 P 850 4900
-F 0 "#PWR022" H 850 4750 50  0001 C CNN
+F 0 "#PWR020" H 850 4750 50  0001 C CNN
 F 1 "VCC" H 850 5050 50  0000 C CNN
 F 2 "" H 850 4900 50  0001 C CNN
@@
 $EndComp
 $Comp
-L GND #PWR023
+L GND #PWR021
 U 1 1 58E02F25
 P 6200 1950
-F 0 "#PWR023" H 6200 1700 50  0001 C CNN
+F 0 "#PWR021" H 6200 1700 50  0001 C CNN
 F 1 "GND" H 6200 1800 50  0000 C CNN
 F 2 "" H 6200 1950 50  0001 C CNN
@@
 $EndComp
 $Comp
-L GND #PWR024
+L GND #PWR022
 U 1 1 58E02F54
 P 6200 2050
-F 0 "#PWR024" H 6200 1800 50  0001 C CNN
+F 0 "#PWR022" H 6200 1800 50  0001 C CNN
 F 1 "GND" H 6200 1900 50  0000 C CNN
 F 2 "" H 6200 2050 50  0001 C CNN
@@
 Text Label 5850 2150 0    60   ~ 0
 3V3
+$Comp
+L CONN_01X01 J6
+U 1 1 58E096FD
+P 4100 5100
+F 0 "J6" H 4100 5200 50  0000 C CNN
+F 1 "CONN_01X01" V 4200 5100 50  0000 C CNN
+F 2 "" H 4100 5100 50  0001 C CNN
+F 3 "" H 4100 5100 50  0001 C CNN
+	1    4100 5100
+	1    0    0    -1
+$EndComp
+$Comp
+L CONN_01X14 J7
+U 1 1 58E0990E
+P 5400 5500
+F 0 "J7" H 5400 6250 50  0000 C CNN
+F 1 "CONN_01X14" V 5500 5500 50  0000 C CNN
+F 2 "" H 5400 5500 50  0001 C CNN
+F 3 "" H 5400 5500 50  0001 C CNN
+	1    5400 5500
+	1    0    0    -1
+$EndComp
+Text Label 3900 2700 0    60   ~ 0
+P37
+Text Label 3900 3000 0    60   ~ 0
+P35
+Text Label 3900 3150 0    60   ~ 0
+P34
+Text Label 3900 3450 0    60   ~ 0
+P32
+Text Label 3900 3750 0    60   ~ 0
+P30
+Text Label 3900 2850 0    60   ~ 0
+P36
+Text Label 3900 3300 0    60   ~ 0
+P33
+Text Label 3900 3600 0    60   ~ 0
+P31
+Text Label 3900 3900 0    60   ~ 0
+P29
+Text Label 3900 4050 0    60   ~ 0
+P28
+Text Label 3900 4200 0    60   ~ 0
+P27
+Text Label 3900 4500 0    60   ~ 0
+P25
+Text Label 3900 4950 0    60   ~ 0
+P22
+NoConn ~ 3900 4650
+Text Label 5200 4850 2    60   ~ 0
+P37
+Text Label 5200 4950 2    60   ~ 0
+P36
+Text Label 5200 5050 2    60   ~ 0
+P35
+Text Label 5200 5150 2    60   ~ 0
+P34
+Text Label 5200 5250 2    60   ~ 0
+P33
+Text Label 5200 5350 2    60   ~ 0
+P32
+Text Label 5200 5450 2    60   ~ 0
+P31
+Text Label 5200 5550 2    60   ~ 0
+P30
+Text Label 5200 5650 2    60   ~ 0
+P29
+Text Label 5200 5750 2    60   ~ 0
+P28
+Text Label 5200 5850 2    60   ~ 0
+P27
+Text Label 5200 6050 2    60   ~ 0
+P25
+Text Label 5200 6150 2    60   ~ 0
+P22
+Text Label 3900 4350 0    60   ~ 0
+P26
+Text Label 5200 5950 2    60   ~ 0
+P26
+Text Label 8400 3800 0    60   ~ 0
+P26
+$Comp
+L PWR_FLAG #FLG023
+U 1 1 58E0A7A9
+P 3900 5100
+F 0 "#FLG023" H 3900 5175 50  0001 C CNN
+F 1 "PWR_FLAG" V 3900 5250 50  0000 L CNN
+F 2 "" H 3900 5100 50  0001 C CNN
+F 3 "" H 3900 5100 50  0001 C CNN
+	1    3900 5100
+	-1   0    0    1
+$EndComp
 $EndSCHEMATC

Commit message: version 0.1
Parts:
- added J8: CONN_01X05, Socket_Strips:Socket_Strip_Straight_1x16_Pitch2.54mm, symbol CONN_01X05
- added J9: CONN_01X05, Socket_Strips:Socket_Strip_Straight_1x05_Pitch2.54mm, symbol CONN_01X05
- J6: footprint (none) -> Pin_Headers:Pin_Header_Straight_1x01_Pitch2.54mm
- J7: footprint (none) -> Socket_Strips:Socket_Strip_Straight_1x14_Pitch2.54mm
Connections:
- net 3V3: now also J9.1 (P1), J9.2 (P2), J9.3 (P3), J9.4 (P4), J9.5 (P5)
- net GND: now also J8.1 (P1), J8.2 (P2), J8.3 (P3), J8.4 (P4), J8.5 (P5)
- net Solar: now reaches D1.2 (A), J2.2
Changed lines of the file:
@@
 NoConn ~ 5800 3700
 NoConn ~ 5800 3800
-Wire Wire Line
-	7750 1900 9100 1900
-Wire Wire Line
-	3900 3600 4700 3600
-Wire Wire Line
-	4700 3600 4700 3550
-Wire Wire Line
-	4700 3850 4350 3850
-Wire Wire Line
-	4350 3850 4350 3150
-Wire Wire Line
-	4350 3150 3900 3150
-Wire Wire Line
-	5800 3300 6150 3300
-Wire Wire Line
-	6150 3300 6150 4450
-Wire Wire Line
-	6150 4450 4400 4450
-Wire Wire Line
-	4400 4450 4400 4050
-Wire Wire Line
-	4400 4050 3900 4050
-Wire Wire Line
-	5800 3400 6000 3400
-Wire Wire Line
-	6000 3400 6000 6500
-Wire Wire Line
-	6000 6500 1100 6500
-Wire Wire Line
-	1100 6500 1100 2050
-Wire Wire Line
-	1100 4050 1800 4050
-Wire Wire Line
-	8400 3800 8900 3800
-Connection ~ 8900 3800
-Connection ~ 8800 1900
-Wire Wire Line
-	8800 1900 8800 2250
-Wire Wire Line
-	8800 2850 9100 2850
-Wire Wire Line
-	7550 4750 8850 4750
-Connection ~ 9000 2850
-Wire Wire Line
-	8800 2850 8800 2550
-Wire Wire Line
-	3900 3300 4200 3300
-Wire Wire Line
-	4200 3300 4200 3350
-Wire Wire Line
-	4200 3350 4700 3350
-Wire Wire Line
-	4700 3450 3900 3450
-Wire Wire Line
-	1700 4950 1800 4950
 Text Label 1550 5100 3    60   ~ 0
 3V3
-Wire Wire Line
-	3900 2550 5250 2550
-Wire Wire Line
-	5250 2550 5250 2950
 Text Label 4550 2550 0    60   ~ 0
 3V3
-Wire Wire Line
-	4700 3650 4700 3750
-Wire Wire Line
-	4700 3750 3900 3750
-Connection ~ 5000 2550
-Connection ~ 4400 2550
-Connection ~ 4800 2550
-Wire Wire Line
-	4400 2550 4400 2100
-Wire Wire Line
-	4800 2100 4800 2550
 $Comp
 L GND #PWR015
@@
 	-1   0    0    1
 $EndComp
-Wire Wire Line
-	1800 4650 850  4650
-Wire Wire Line
-	850  4650 850  2450
-Wire Wire Line
-	1800 4500 900  4500
-Wire Wire Line
-	900  4500 900  2350
-Wire Wire Line
-	900  2350 850  2350
-Wire Wire Line
-	1800 4350 950  4350
-Wire Wire Line
-	950  4350 950  2250
-Wire Wire Line
-	950  2250 850  2250
-Wire Wire Line
-	1800 4200 1000 4200
-Wire Wire Line
-	1000 4200 1000 2150
-Wire Wire Line
-	1000 2150 850  2150
-Connection ~ 1100 4050
-Wire Wire Line
-	1100 2050 850  2050
-Wire Wire Line
-	1800 3900 1150 3900
-Wire Wire Line
-	1150 3900 1150 1950
-Wire Wire Line
-	1150 1950 850  1950
-Wire Wire Line
-	1800 3750 1200 3750
-Wire Wire Line
-	1200 3750 1200 1850
-Wire Wire Line
-	1200 1850 850  1850
-Wire Wire Line
-	1800 3600 1250 3600
-Wire Wire Line
-	1250 3600 1250 1750
-Wire Wire Line
-	1250 1750 850  1750
-Wire Wire Line
-	1800 3450 1300 3450
-Wire Wire Line
-	1300 3450 1300 1650
-Wire Wire Line
-	1300 1650 850  1650
-Wire Wire Line
-	1800 3300 1350 3300
-Wire Wire Line
-	1350 3300 1350 1550
-Wire Wire Line
-	1350 1550 850  1550
-Wire Wire Line
-	1400 1450 1400 3150
-Wire Wire Line
-	850  1450 1400 1450
-Wire Wire Line
-	850  1350 1450 1350
-Wire Wire Line
-	1450 1350 1450 3000
-Wire Wire Line
-	1450 3000 1800 3000
-Wire Wire Line
-	1800 2850 1500 2850
-Wire Wire Line
-	1500 2850 1500 1250
-Wire Wire Line
-	1500 1250 850  1250
-Wire Wire Line
-	850  1150 1550 1150
-Wire Wire Line
-	1550 1150 1550 2700
-Wire Wire Line
-	1550 2700 1800 2700
-Wire Wire Line
-	1800 2550 1600 2550
-Wire Wire Line
-	1600 2550 1600 1050
-Wire Wire Line
-	1600 1050 850  1050
-Wire Wire Line
-	850  950  1650 950
-Wire Wire Line
-	1650 950  1650 2400
-Wire Wire Line
-	1650 2400 1800 2400
-Wire Wire Line
-	1800 2250 1700 2250
-Wire Wire Line
-	1700 2250 1700 850
-Wire Wire Line
-	1700 850  850  850
 $Comp
 L CONN_01X03 J4
@@
 	-1   0    0    1
 $EndComp
-Wire Wire Line
-	850  5100 1800 5100
 $Comp
 L GND #PWR019
@@
 	1    0    0    -1
 $EndComp
-Wire Wire Line
-	1400 3150 1800 3150
 $Comp
 L CONN_01X03 J5
@@
 	0    1    1    0
 $EndComp
-Wire Wire Line
-	5750 2150 6200 2150
 Text Label 5850 2150 0    60   ~ 0
 3V3
@@
 F 0 "J6" H 4100 5200 50  0000 C CNN
 F 1 "CONN_01X01" V 4200 5100 50  0000 C CNN
-F 2 "" H 4100 5100 50  0001 C CNN
+F 2 "Pin_Headers:Pin_Header_Straight_1x01_Pitch2.54mm" H 4100 5100 50  0001 C CNN
 F 3 "" H 4100 5100 50  0001 C CNN
 	1    4100 5100
@@
 F 0 "J7" H 5400 6250 50  0000 C CNN
 F 1 "CONN_01X14" V 5500 5500 50  0000 C CNN
-F 2 "" H 5400 5500 50  0001 C CNN
+F 2 "Socket_Strips:Socket_Strip_Straight_1x14_Pitch2.54mm" H 5400 5500 50  0001 C CNN
 F 3 "" H 5400 5500 50  0001 C CNN
 	1    5400 5500
@@
 	-1   0    0    1
 $EndComp
+Text Label 8800 2850 2    60   ~ 0
+Solar
+$Comp
+L CONN_01X05 J8
+U 1 1 58E0ADB1
+P 3150 7150
+F 0 "J8" H 3150 7450 50  0000 C CNN
+F 1 "CONN_01X05" V 3250 7150 50  0000 C CNN
+F 2 "Socket_Strips:Socket_Strip_Straight_1x16_Pitch2.54mm" H 3150 7150 50  0001 C CNN
+F 3 "" H 3150 7150 50  0001 C CNN
+	1    3150 7150
+	1    0    0    -1
+$EndComp
+Wire Wire Line
+	7750 1900 9100 1900
+Wire Wire Line
+	3900 3600 4700 3600
+Wire Wire Line
+	4700 3600 4700 3550
+Wire Wire Line
+	4700 3850 4350 3850
+Wire Wire Line
+	4350 3850 4350 3150
+Wire Wire Line
+	4350 3150 3900 3150
+Wire Wire Line
+	5800 3300 6150 3300
+Wire Wire Line
+	6150 3300 6150 4450
+Wire Wire Line
+	6150 4450 4400 4450
+Wire Wire Line
+	4400 4450 4400 4050
+Wire Wire Line
+	4400 4050 3900 4050
+Wire Wire Line
+	5800 3400 6000 3400
+Wire Wire Line
+	6000 3400 6000 6500
+Wire Wire Line
+	6000 6500 1100 6500
+Wire Wire Line
+	1100 6500 1100 2050
+Wire Wire Line
+	1100 4050 1800 4050
+Wire Wire Line
+	8400 3800 8900 3800
+Connection ~ 8900 3800
+Connection ~ 8800 1900
+Wire Wire Line
+	8800 1900 8800 2250
+Wire Wire Line
+	8800 2850 9100 2850
+Wire Wire Line
+	7550 4750 8850 4750
+Connection ~ 9000 2850
+Wire Wire Line
+	8800 2850 8800 2550
+Wire Wire Line
+	3900 3300 4200 3300
+Wire Wire Line
+	4200 3300 4200 3350
+Wire Wire Line
+	4200 3350 4700 3350
+Wire Wire Line
+	4700 3450 3900 3450
+Wire Wire Line
+	1700 4950 1800 4950
+Wire Wire Line
+	3900 2550 5250 2550
+Wire Wire Line
+	5250 2550 5250 2950
+Wire Wire Line
+	4700 3650 4700 3750
+Wire Wire Line
+	4700 3750 3900 3750
+Connection ~ 5000 2550
+Connection ~ 4400 2550
+Connection ~ 4800 2550
+Wire Wire Line
+	4400 2550 4400 2100
+Wire Wire Line
+	4800 2100 4800 2550
+Wire Wire Line
+	1800 4650 850  4650
+Wire Wire Line
+	850  4650 850  2450
+Wire Wire Line
+	1800 4500 900  4500
+Wire Wire Line
+	900  4500 900  2350
+Wire Wire Line
+	900  2350 850  2350
+Wire Wire Line
+	1800 4350 950  4350
+Wire Wire Line
+	950  4350 950  2250
+Wire Wire Line
+	950  2250 850  2250
+Wire Wire Line
+	1800 4200 1000 4200
+Wire Wire Line
+	1000 4200 1000 2150
+Wire Wire Line
+	1000 2150 850  2150
+Connection ~ 1100 4050
+Wire Wire Line
+	1100 2050 850  2050
+Wire Wire Line
+	1800 3900 1150 3900
+Wire Wire Line
+	1150 3900 1150 1950
+Wire Wire Line
+	1150 1950 850  1950
+Wire Wire Line
+	1800 3750 1200 3750
+Wire Wire Line
+	1200 3750 1200 1850
+Wire Wire Line
+	1200 1850 850  1850
+Wire Wire Line
+	1800 3600 1250 3600
+Wire Wire Line
+	1250 3600 1250 1750
+Wire Wire Line
+	1250 1750 850  1750
+Wire Wire Line
+	1800 3450 1300 3450
+Wire Wire Line
+	1300 3450 1300 1650
+Wire Wire Line
+	1300 1650 850  1650
+Wire Wire Line
+	1800 3300 1350 3300
+Wire Wire Line
+	1350 3300 1350 1550
+Wire Wire Line
+	1350 1550 850  1550
+Wire Wire Line
+	1400 1450 1400 3150
+Wire Wire Line
+	850  1450 1400 1450
+Wire Wire Line
+	850  1350 1450 1350
+Wire Wire Line
+	1450 1350 1450 3000
+Wire Wire Line
+	1450 3000 1800 3000
+Wire Wire Line
+	1800 2850 1500 2850
+Wire Wire Line
+	1500 2850 1500 1250
+Wire Wire Line
+	1500 1250 850  1250
+Wire Wire Line
+	850  1150 1550 1150
+Wire Wire Line
+	1550 1150 1550 2700
+Wire Wire Line
+	1550 2700 1800 2700
+Wire Wire Line
+	1800 2550 1600 2550
+Wire Wire Line
+	1600 2550 1600 1050
+Wire Wire Line
+	1600 1050 850  1050
+Wire Wire Line
+	850  950  1650 950
+Wire Wire Line
+	1650 950  1650 2400
+Wire Wire Line
+	1650 2400 1800 2400
+Wire Wire Line
+	1800 2250 1700 2250
+Wire Wire Line
+	1700 2250 1700 850
+Wire Wire Line
+	1700 850  850  850
+Wire Wire Line
+	850  5100 1800 5100
+Wire Wire Line
+	1400 3150 1800 3150
+Wire Wire Line
+	5750 2150 6200 2150
+Wire Wire Line
+	2950 6950 2950 7350
+Connection ~ 2950 7050
+Connection ~ 2950 7150
+Connection ~ 2950 7250
+$Comp
+L GND #PWR024
+U 1 1 58E0B20A
+P 2950 7350
+F 0 "#PWR024" H 2950 7100 50  0001 C CNN
+F 1 "GND" H 2950 7200 50  0000 C CNN
+F 2 "" H 2950 7350 50  0001 C CNN
+F 3 "" H 2950 7350 50  0001 C CNN
+	1    2950 7350
+	1    0    0    -1
+$EndComp
+$Comp
+L CONN_01X05 J9
+U 1 1 58E0B40A
+P 3700 7150
+F 0 "J9" H 3700 7450 50  0000 C CNN
+F 1 "CONN_01X05" V 3800 7150 50  0000 C CNN
+F 2 "Socket_Strips:Socket_Strip_Straight_1x05_Pitch2.54mm" H 3700 7150 50  0001 C CNN
+F 3 "" H 3700 7150 50  0001 C CNN
+	1    3700 7150
+	1    0    0    -1
+$EndComp
+Wire Wire Line
+	3500 6950 3500 7350
+Connection ~ 3500 7050
+Connection ~ 3500 7150
+Connection ~ 3500 7250
+Text Label 3500 7350 3    60   ~ 0
+3V3
 $EndSCHEMATC

Commit message: 0.1 version sent to production
Parts:
- J8: footprint Socket_Strips:Socket_Strip_Straight_1x16_Pitch2.54mm -> Socket_Strips:Socket_Strip_Straight_1x05_Pitch2.54mm
Changed lines of the file:
@@
 F 0 "J8" H 3150 7450 50  0000 C CNN
 F 1 "CONN_01X05" V 3250 7150 50  0000 C CNN
-F 2 "Socket_Strips:Socket_Strip_Straight_1x16_Pitch2.54mm" H 3150 7150 50  0001 C CNN
+F 2 "Socket_Strips:Socket_Strip_Straight_1x05_Pitch2.54mm" H 3150 7150 50  0001 C CNN
 F 3 "" H 3150 7150 50  0001 C CNN
 	1    3150 7150
