File: AVR-LORA.sch (KiCad schematic (older format))
At the start: 22 parts, among them J1 Batt, J2 Solar

Commit message: Add AVR pull ups
Parts:
- added R? (x2): 4K7, symbol Device:R
Connections:
- net labels removed: P26
Other:
- note added: "I2C pull ups"
- moved on the sheet: C?
Changed lines of the file:
@@
 $EndComp
 Text Label 8150 3550 1    60   ~ 0
-P26
+D1
 Text Label 8000 2150 2    60   ~ 0
 Solar
@@
 L Regulator_Linear:MCP1700-3302E_SOT23 U?
 U 1 1 611E964D
-P 2350 1200
-F 0 "U?" H 2350 1442 50  0000 C CNN
-F 1 "MCP1700-3302E_SOT23" H 2350 1351 50  0000 C CNN
-F 2 "Package_TO_SOT_SMD:SOT-23" H 2350 1425 50  0001 C CNN
-F 3 "http://ww1.microchip.com/downloads/en/DeviceDoc/20001826D.pdf" H 2350 1200 50  0001 C CNN
-	1    2350 1200
+P 2350 1050
+F 0 "U?" H 2350 1292 50  0000 C CNN
+F 1 "MCP1700-3302E_SOT23" H 2350 1201 50  0000 C CNN
+F 2 "Package_TO_SOT_SMD:SOT-23" H 2350 1275 50  0001 C CNN
+F 3 "http://ww1.microchip.com/downloads/en/DeviceDoc/20001826D.pdf" H 2350 1050 50  0001 C CNN
+	1    2350 1050
 	1    0    0    -1
 $EndComp
@@
 L power:GND #PWR?
 U 1 1 611E9B95
-P 2350 1500
-F 0 "#PWR?" H 2350 1250 50  0001 C CNN
-F 1 "GND" H 2350 1350 50  0000 C CNN
-F 2 "" H 2350 1500 50  0000 C CNN
-F 3 "" H 2350 1500 50  0000 C CNN
-	1    2350 1500
-	1    0    0    -1
-$EndComp
-Text Label 2800 1200 0    60   ~ 0
+P 2350 1350
+F 0 "#PWR?" H 2350 1100 50  0001 C CNN
+F 1 "GND" H 2350 1200 50  0000 C CNN
+F 2 "" H 2350 1350 50  0000 C CNN
+F 3 "" H 2350 1350 50  0000 C CNN
+	1    2350 1350
+	1    0    0    -1
+$EndComp
+Text Label 2800 1050 0    60   ~ 0
 3V3
 $Comp
 L power:VCC #PWR?
 U 1 1 611EA431
-P 1850 1200
-F 0 "#PWR?" H 1850 1050 50  0001 C CNN
-F 1 "VCC" H 1850 1350 50  0000 C CNN
-F 2 "" H 1850 1200 50  0000 C CNN
-F 3 "" H 1850 1200 50  0000 C CNN
-	1    1850 1200
+P 1850 1050
+F 0 "#PWR?" H 1850 900 50  0001 C CNN
+F 1 "VCC" H 1850 1200 50  0000 C CNN
+F 2 "" H 1850 1050 50  0000 C CNN
+F 3 "" H 1850 1050 50  0000 C CNN
+	1    1850 1050
 	0    -1   -1   0
 $EndComp
@@
 L STM-LORA-rescue:C C?
 U 1 1 611EB9C7
-P 2700 1350
-F 0 "C?" H 2725 1450 50  0000 L CNN
-F 1 "1uF" H 2725 1250 50  0000 L CNN
-F 2 "Capacitors_THT:C_Disc_D5.0mm_W2.5mm_P5.00mm" H 2738 1200 50  0001 C CNN
-F 3 "" H 2700 1350 50  0000 C CNN
-	1    2700 1350
+P 2700 1200
+F 0 "C?" H 2725 1300 50  0000 L CNN
+F 1 "1uF" H 2725 1100 50  0000 L CNN
+F 2 "Capacitors_THT:C_Disc_D5.0mm_W2.5mm_P5.00mm" H 2738 1050 50  0001 C CNN
+F 3 "" H 2700 1200 50  0000 C CNN
+	1    2700 1200
 	1    0    0    -1
 $EndComp
@@
 L STM-LORA-rescue:C C?
 U 1 1 611EC9E6
-P 2000 1350
-F 0 "C?" H 2025 1450 50  0000 L CNN
-F 1 "1uF" H 2025 1250 50  0000 L CNN
-F 2 "Capacitors_THT:C_Disc_D5.0mm_W2.5mm_P5.00mm" H 2038 1200 50  0001 C CNN
-F 3 "" H 2000 1350 50  0000 C CNN
-	1    2000 1350
-	1    0    0    -1
-$EndComp
-Wire Wire Line
-	2650 1200 2700 1200
-Wire Wire Line
-	2700 1200 2800 1200
-Connection ~ 2700 1200
-Wire Wire Line
-	1850 1200 2000 1200
-Wire Wire Line
-	2000 1200 2050 1200
-Connection ~ 2000 1200
-Wire Wire Line
-	2000 1500 2350 1500
-Connection ~ 2350 1500
-Wire Wire Line
-	2350 1500 2700 1500
+P 2000 1200
+F 0 "C?" H 2025 1300 50  0000 L CNN
+F 1 "1uF" H 2025 1100 50  0000 L CNN
+F 2 "Capacitors_THT:C_Disc_D5.0mm_W2.5mm_P5.00mm" H 2038 1050 50  0001 C CNN
+F 3 "" H 2000 1200 50  0000 C CNN
+	1    2000 1200
+	1    0    0    -1
+$EndComp
+Wire Wire Line
+	2650 1050 2700 1050
+Wire Wire Line
+	2700 1050 2800 1050
+Connection ~ 2700 1050
+Wire Wire Line
+	1850 1050 2000 1050
+Wire Wire Line
+	2000 1050 2050 1050
+Connection ~ 2000 1050
+Wire Wire Line
+	2000 1350 2350 1350
+Connection ~ 2350 1350
+Wire Wire Line
+	2350 1350 2700 1350
 $Comp
 L RFM95:RFM95HW U?
@@
 L Jumper:SolderJumper_2_Open JP?
 U 1 1 61210DFF
-P 5600 1750
-F 0 "JP?" H 5600 1955 50  0000 C CNN
-F 1 "SolderJumper_2_Open" H 5600 1600 50  0000 C CNN
-F 2 "" H 5600 1750 50  0001 C CNN
-F 3 "~" H 5600 1750 50  0001 C CNN
-	1    5600 1750
-	1    0    0    -1
-$EndComp
-Text Label 5750 1750 0    60   ~ 0
+P 2350 1800
+F 0 "JP?" H 2350 1950 50  0000 C CNN
+F 1 "SolderJumper_2_Open" H 2350 1650 50  0000 C CNN
+F 2 "" H 2350 1800 50  0001 C CNN
+F 3 "~" H 2350 1800 50  0001 C CNN
+	1    2350 1800
+	1    0    0    -1
+$EndComp
+Text Label 2500 1800 0    60   ~ 0
 3V3
 $Comp
 L power:VCC #PWR?
 U 1 1 61211C58
-P 5450 1750
-F 0 "#PWR?" H 5450 1600 50  0001 C CNN
-F 1 "VCC" H 5450 1900 50  0000 C CNN
-F 2 "" H 5450 1750 50  0000 C CNN
-F 3 "" H 5450 1750 50  0000 C CNN
-	1    5450 1750
+P 2200 1800
+F 0 "#PWR?" H 2200 1650 50  0001 C CNN
+F 1 "VCC" H 2200 1950 50  0000 C CNN
+F 2 "" H 2200 1800 50  0000 C CNN
+F 3 "" H 2200 1800 50  0000 C CNN
+	1    2200 1800
 	0    -1   -1   0
 $EndComp
@@
 Text Label 7250 6050 2    50   ~ 0
 D7
+$Comp
+L Device:R R?
+U 1 1 612233E5
+P 6750 3000
+F 0 "R?" H 6820 3046 50  0000 L CNN
+F 1 "4K7" H 6820 2955 50  0000 L CNN
+F 2 "" V 6680 3000 50  0001 C CNN
+F 3 "~" H 6750 3000 50  0001 C CNN
+	1    6750 3000
+	1    0    0    -1
+$EndComp
+$Comp
+L Device:R R?
+U 1 1 6122370A
+P 7100 3000
+F 0 "R?" H 7170 3046 50  0000 L CNN
+F 1 "4K7" H 7170 2955 50  0000 L CNN
+F 2 "" V 7030 3000 50  0001 C CNN
+F 3 "~" H 7100 3000 50  0001 C CNN
+	1    7100 3000
+	1    0    0    -1
+$EndComp
+Text Label 6750 2850 1    60   ~ 0
+3V3
+Text Label 7100 2850 1    60   ~ 0
+3V3
+Text Label 6750 3150 3    50   ~ 0
+A3
+Text Label 7100 3150 3    50   ~ 0
+A2
+Text Notes 6700 3400 0    50   ~ 0
+I2C pull ups
 $EndSCHEMATC

Commit message: Add AVR crystals
Parts:
- added C10, C11, C12, C9: 12pF, symbol Device:C
- added JP2, JP3, JP4, JP5: SolderJumper_2_Open, symbol Jumper:SolderJumper_2_Open
- added Y1, Y2: Crystal, symbol Device:Crystal
- gave numbers to parts that had none: 19
Connections:
- net labels added: CA0, CA1, CF0, CF1
- wire segments 33 -> 49
Other:
- note added: "Optional external crystals"
- moved on the sheet: R4

Commit message: Add footprints to AVR
Parts:
- C1, C2, C3, C4, C5, C6, C7, C8: footprint Capacitors_THT:C_Disc_D5.0mm_W2.5mm_P5.00mm -> Capacitor_SMD:C_1206_3216Metric
- C10, C9: value 12pF -> 22pF; footprint (none) -> Capacitor_SMD:C_1206_3216Metric
- C11, C12: value 12pF -> 10pF; footprint (none) -> Capacitor_SMD:C_1206_3216Metric
- D1: value BAT85 -> BAT54S; footprint Diodes_THT:D_DO-35_SOD27_P2.54mm_Vertical_AnodeUp -> Diode_SMD:D_SOT-23_ANK
- D2: footprint (none) -> LED_SMD:LED_1206_3216Metric
- J1, J2: footprint Pin_Headers:Pin_Header_Straight_1x02_Pitch2.54mm -> Connector_PinHeader_2.54mm:PinHeader_1x02_P2.54mm_Vertical
- J3: footprint Pin_Headers:Pin_Header_Straight_1x01_Pitch2.54mm -> Connector_PinHeader_2.54mm:PinHeader_1x01_P2.54mm_Vertical
- J4, J5: footprint Socket_Strips:Socket_Strip_Straight_1x14_Pitch2.54mm -> Connector_PinHeader_2.54mm:PinHeader_1x14_P2.54mm_Vertical
- JP1, JP2, JP3, JP4, JP5: footprint (none) -> Jumper:SolderJumper-2_P1.3mm_Open_Pad1.0x1.5mm
- R1, R2: footprint Resistors_THT:R_Axial_DIN0309_L9.0mm_D3.2mm_P2.54mm_Vertical -> Resistor_SMD:R_1206_3216Metric
- R3, R4, R5: footprint (none) -> Resistor_SMD:R_1206_3216Metric
- Y1: value Crystal -> 8MHz; footprint (none) -> Crystal:Crystal_SMD_MicroCrystal_CC7V-T1A-2Pin_3.2x1.5mm
- Y2: value Crystal -> 32768Hz; footprint (none) -> Crystal:Crystal_SMD_MicroCrystal_CC7V-T1A-2Pin_3.2x1.5mm
Changed lines of the file:
@@
 F 0 "R2" V 8380 3050 50  0000 C CNN
 F 1 "100k" V 8300 3050 50  0000 C CNN
-F 2 "Resistors_THT:R_Axial_DIN0309_L9.0mm_D3.2mm_P2.54mm_Vertical" V 8230 3050 50  0001 C CNN
+F 2 "Resistor_SMD:R_1206_3216Metric" V 8230 3050 50  0001 C CNN
 F 3 "" H 8300 3050 50  0000 C CNN
 	1    8300 3050
@@
 F 0 "R1" V 8080 3050 50  0000 C CNN
 F 1 "100k" V 8000 3050 50  0000 C CNN
-F 2 "Resistors_THT:R_Axial_DIN0309_L9.0mm_D3.2mm_P2.54mm_Vertical" V 7930 3050 50  0001 C CNN
+F 2 "Resistor_SMD:R_1206_3216Metric" V 7930 3050 50  0001 C CNN
 F 3 "" H 8000 3050 50  0000 C CNN
 	1    8000 3050
@@
 P 8000 1700
 F 0 "D1" H 8000 1800 50  0000 C CNN
-F 1 "BAT85" H 8000 1600 50  0000 C CNN
-F 2 "Diodes_THT:D_DO-35_SOD27_P2.54mm_Vertical_AnodeUp" H 8000 1700 50  0001 C CNN
+F 1 "BAT54S" H 8000 1600 50  0000 C CNN
+F 2 "Diode_SMD:D_SOT-23_ANK" H 8000 1700 50  0001 C CNN
 F 3 "" H 8000 1700 50  0000 C CNN
 	1    8000 1700
@@
 F 0 "J1" H 8600 1475 50  0000 C CNN
 F 1 "Batt" H 8600 1100 50  0000 C CNN
-F 2 "Pin_Headers:Pin_Header_Straight_1x02_Pitch2.54mm" H 8600 1400 50  0001 C CNN
+F 2 "Connector_PinHeader_2.54mm:PinHeader_1x02_P2.54mm_Vertical" H 8600 1400 50  0001 C CNN
 F 3 "" H 8600 1400 50  0001 C CNN
 	1    8600 1300
@@
 F 0 "J2" H 8600 2425 50  0000 C CNN
 F 1 "Solar" H 8600 2050 50  0000 C CNN
-F 2 "Pin_Headers:Pin_Header_Straight_1x02_Pitch2.54mm" H 8600 2350 50  0001 C CNN
+F 2 "Connector_PinHeader_2.54mm:PinHeader_1x02_P2.54mm_Vertical" H 8600 2350 50  0001 C CNN
 F 3 "" H 8600 2350 50  0001 C CNN
 	1    8600 2250
@@
 F 0 "J4" H 7450 6250 50  0000 C CNN
 F 1 "CONN_01X14" V 7550 5500 50  0000 C CNN
-F 2 "Socket_Strips:Socket_Strip_Straight_1x14_Pitch2.54mm" H 7450 5500 50  0001 C CNN
+F 2 "Connector_PinHeader_2.54mm:PinHeader_1x14_P2.54mm_Vertical" H 7450 5500 50  0001 C CNN
 F 3 "" H 7450 5500 50  0001 C CNN
 	1    7450 5500
@@
 F 0 "J3" H 4700 3050 50  0000 C CNN
 F 1 "CONN_01X01" V 4800 2950 50  0000 C CNN
-F 2 "Pin_Headers:Pin_Header_Straight_1x01_Pitch2.54mm" H 4700 2950 50  0001 C CNN
+F 2 "Connector_PinHeader_2.54mm:PinHeader_1x01_P2.54mm_Vertical" H 4700 2950 50  0001 C CNN
 F 3 "" H 4700 2950 50  0001 C CNN
 	1    4700 2950
@@
 F 0 "C7" H 3525 2600 50  0000 L CNN
 F 1 "100nF" H 3525 2400 50  0000 L CNN
-F 2 "Capacitors_THT:C_Disc_D5.0mm_W2.5mm_P5.00mm" H 3538 2350 50  0001 C CNN
+F 2 "Capacitor_SMD:C_1206_3216Metric" H 3538 2350 50  0001 C CNN
 F 3 "" H 3500 2500 50  0000 C CNN
 	1    3500 2500
@@
 F 0 "C8" H 3825 2600 50  0000 L CNN
 F 1 "1uF" H 3825 2400 50  0000 L CNN
-F 2 "Capacitors_THT:C_Disc_D5.0mm_W2.5mm_P5.00mm" H 3838 2350 50  0001 C CNN
+F 2 "Capacitor_SMD:C_1206_3216Metric" H 3838 2350 50  0001 C CNN
 F 3 "" H 3800 2500 50  0000 C CNN
 	1    3800 2500
@@
 F 0 "C5" H 2925 2600 50  0000 L CNN
 F 1 "100nF" H 2925 2400 50  0000 L CNN
-F 2 "Capacitors_THT:C_Disc_D5.0mm_W2.5mm_P5.00mm" H 2938 2350 50  0001 C CNN
+F 2 "Capacitor_SMD:C_1206_3216Metric" H 2938 2350 50  0001 C CNN
 F 3 "" H 2900 2500 50  0000 C CNN
 	1    2900 2500
@@
 F 0 "C6" H 3225 2600 50  0000 L CNN
 F 1 "1uF" H 3225 2400 50  0000 L CNN
-F 2 "Capacitors_THT:C_Disc_D5.0mm_W2.5mm_P5.00mm" H 3238 2350 50  0001 C CNN
+F 2 "Capacitor_SMD:C_1206_3216Metric" H 3238 2350 50  0001 C CNN
 F 3 "" H 3200 2500 50  0000 C CNN
 	1    3200 2500
@@
 F 0 "C2" H 2325 2600 50  0000 L CNN
 F 1 "100nF" H 2325 2400 50  0000 L CNN
-F 2 "Capacitors_THT:C_Disc_D5.0mm_W2.5mm_P5.00mm" H 2338 2350 50  0001 C CNN
+F 2 "Capacitor_SMD:C_1206_3216Metric" H 2338 2350 50  0001 C CNN
 F 3 "" H 2300 2500 50  0000 C CNN
 	1    2300 2500
@@
 F 0 "C3" H 2625 2600 50  0000 L CNN
 F 1 "1uF" H 2625 2400 50  0000 L CNN
-F 2 "Capacitors_THT:C_Disc_D5.0mm_W2.5mm_P5.00mm" H 2638 2350 50  0001 C CNN
+F 2 "Capacitor_SMD:C_1206_3216Metric" H 2638 2350 50  0001 C CNN
 F 3 "" H 2600 2500 50  0000 C CNN
 	1    2600 2500
@@
 F 0 "C4" H 2725 1300 50  0000 L CNN
 F 1 "1uF" H 2725 1100 50  0000 L CNN
-F 2 "Capacitors_THT:C_Disc_D5.0mm_W2.5mm_P5.00mm" H 2738 1050 50  0001 C CNN
+F 2 "Capacitor_SMD:C_1206_3216Metric" H 2738 1050 50  0001 C CNN
 F 3 "" H 2700 1200 50  0000 C CNN
 	1    2700 1200
@@
 F 0 "C1" H 2025 1300 50  0000 L CNN
 F 1 "1uF" H 2025 1100 50  0000 L CNN
-F 2 "Capacitors_THT:C_Disc_D5.0mm_W2.5mm_P5.00mm" H 2038 1050 50  0001 C CNN
+F 2 "Capacitor_SMD:C_1206_3216Metric" H 2038 1050 50  0001 C CNN
 F 3 "" H 2000 1200 50  0000 C CNN
 	1    2000 1200
@@
 F 0 "JP1" H 2350 1950 50  0000 C CNN
 F 1 "SolderJumper_2_Open" H 2350 1650 50  0000 C CNN
-F 2 "" H 2350 1800 50  0001 C CNN
+F 2 "Jumper:SolderJumper-2_P1.3mm_Open_Pad1.0x1.5mm" H 2350 1800 50  0001 C CNN
 F 3 "~" H 2350 1800 50  0001 C CNN
 	1    2350 1800
@@
 F 0 "D2" V 6939 1782 50  0000 R CNN
 F 1 "LED" V 6848 1782 50  0000 R CNN
-F 2 "" H 6900 1900 50  0001 C CNN
+F 2 "LED_SMD:LED_1206_3216Metric" H 6900 1900 50  0001 C CNN
 F 3 "~" H 6900 1900 50  0001 C CNN
 	1    6900 1900
@@
 F 0 "R4" H 6970 1646 50  0000 L CNN
 F 1 "100R" H 6970 1555 50  0000 L CNN
-F 2 "" V 6830 1600 50  0001 C CNN
+F 2 "Resistor_SMD:R_1206_3216Metric" V 6830 1600 50  0001 C CNN
 F 3 "~" H 6900 1600 50  0001 C CNN
 	1    6900 1600
@@
 F 0 "J5" H 8450 6250 50  0000 C CNN
 F 1 "CONN_01X14" V 8550 5500 50  0000 C CNN
-F 2 "Socket_Strips:Socket_Strip_Straight_1x14_Pitch2.54mm" H 8450 5500 50  0001 C CNN
+F 2 "Connector_PinHeader_2.54mm:PinHeader_1x14_P2.54mm_Vertical" H 8450 5500 50  0001 C CNN
 F 3 "" H 8450 5500 50  0001 C CNN
 	1    8450 5500
@@
 F 0 "R3" H 6820 3046 50  0000 L CNN
 F 1 "4K7" H 6820 2955 50  0000 L CNN
-F 2 "" V 6680 3000 50  0001 C CNN
+F 2 "Resistor_SMD:R_1206_3216Metric" V 6680 3000 50  0001 C CNN
 F 3 "~" H 6750 3000 50  0001 C CNN
 	1    6750 3000
@@
 F 0 "R5" H 7170 3046 50  0000 L CNN
 F 1 "4K7" H 7170 2955 50  0000 L CNN
-F 2 "" V 7030 3000 50  0001 C CNN
+F 2 "Resistor_SMD:R_1206_3216Metric" V 7030 3000 50  0001 C CNN
 F 3 "~" H 7100 3000 50  0001 C CNN
 	1    7100 3000
@@
 P 4300 1400
 F 0 "Y1" H 4300 1668 50  0000 C CNN
-F 1 "Crystal" H 4300 1577 50  0000 C CNN
-F 2 "" H 4300 1400 50  0001 C CNN
+F 1 "8MHz" H 4300 1577 50  0000 C CNN
+F 2 "Crystal:Crystal_SMD_MicroCrystal_CC7V-T1A-2Pin_3.2x1.5mm" H 4300 1400 50  0001 C CNN
 F 3 "~" H 4300 1400 50  0001 C CNN
 	1    4300 1400
@@
 P 4500 1650
 F 0 "C10" H 4615 1696 50  0000 L CNN
-F 1 "12pF" H 4615 1605 50  0000 L CNN
-F 2 "" H 4538 1500 50  0001 C CNN
+F 1 "22pF" H 4615 1605 50  0000 L CNN
+F 2 "Capacitor_SMD:C_1206_3216Metric" H 4538 1500 50  0001 C CNN
 F 3 "~" H 4500 1650 50  0001 C CNN
 	1    4500 1650
@@
 P 4100 1650
 F 0 "C9" H 4215 1696 50  0000 L CNN
-F 1 "12pF" H 4215 1605 50  0000 L CNN
-F 2 "" H 4138 1500 50  0001 C CNN
+F 1 "22pF" H 4215 1605 50  0000 L CNN
+F 2 "Capacitor_SMD:C_1206_3216Metric" H 4138 1500 50  0001 C CNN
 F 3 "~" H 4100 1650 50  0001 C CNN
 	1    4100 1650
@@
 F 0 "JP2" H 3950 1017 50  0000 C CNN
 F 1 "SolderJumper_2_Open" V 3995 1218 50  0001 L CNN
-F 2 "" H 3950 1150 50  0001 C CNN
+F 2 "Jumper:SolderJumper-2_P1.3mm_Open_Pad1.0x1.5mm" H 3950 1150 50  0001 C CNN
 F 3 "~" H 3950 1150 50  0001 C CNN
 	1    3950 1150
@@
 F 0 "JP3" H 4650 1263 50  0000 C CNN
 F 1 "SolderJumper_2_Open" V 4695 1218 50  0001 L CNN
-F 2 "" H 4650 1150 50  0001 C CNN
+F 2 "Jumper:SolderJumper-2_P1.3mm_Open_Pad1.0x1.5mm" H 4650 1150 50  0001 C CNN
 F 3 "~" H 4650 1150 50  0001 C CNN
 	1    4650 1150
@@
 P 5800 1400
 F 0 "Y2" H 5800 1668 50  0000 C CNN
-F 1 "Crystal" H 5800 1577 50  0000 C CNN
-F 2 "" H 5800 1400 50  0001 C CNN
+F 1 "32768Hz" H 5800 1577 50  0000 C CNN
+F 2 "Crystal:Crystal_SMD_MicroCrystal_CC7V-T1A-2Pin_3.2x1.5mm" H 5800 1400 50  0001 C CNN
 F 3 "~" H 5800 1400 50  0001 C CNN
 	1    5800 1400
@@
 P 6000 1650
 F 0 "C12" H 6115 1696 50  0000 L CNN
-F 1 "12pF" H 6115 1605 50  0000 L CNN
-F 2 "" H 6038 1500 50  0001 C CNN
+F 1 "10pF" H 6115 1605 50  0000 L CNN
+F 2 "Capacitor_SMD:C_1206_3216Metric" H 6038 1500 50  0001 C CNN
 F 3 "~" H 6000 1650 50  0001 C CNN
 	1    6000 1650
@@
 P 5600 1650
 F 0 "C11" H 5715 1696 50  0000 L CNN
-F 1 "12pF" H 5715 1605 50  0000 L CNN
-F 2 "" H 5638 1500 50  0001 C CNN
+F 1 "10pF" H 5715 1605 50  0000 L CNN
+F 2 "Capacitor_SMD:C_1206_3216Metric" H 5638 1500 50  0001 C CNN
 F 3 "~" H 5600 1650 50  0001 C CNN
 	1    5600 1650
@@
 F 0 "JP4" H 5450 1017 50  0000 C CNN
 F 1 "SolderJumper_2_Open" V 5495 1218 50  0001 L CNN
-F 2 "" H 5450 1150 50  0001 C CNN
+F 2 "Jumper:SolderJumper-2_P1.3mm_Open_Pad1.0x1.5mm" H 5450 1150 50  0001 C CNN
 F 3 "~" H 5450 1150 50  0001 C CNN
 	1    5450 1150
@@
 F 0 "JP5" H 6150 1263 50  0000 C CNN
 F 1 "SolderJumper_2_Open" V 6195 1218 50  0001 L CNN
-F 2 "" H 6150 1150 50  0001 C CNN
+F 2 "Jumper:SolderJumper-2_P1.3mm_Open_Pad1.0x1.5mm" H 6150 1150 50  0001 C CNN
 F 3 "~" H 6150 1150 50  0001 C CNN
 	1    6150 1150

Commit message: Layout AVR
Parts:
- R4: renamed from R1; value 100k -> 1M
- R5: renamed from R2; value 100k -> 1M
- Y1: value 8MHz -> 24MHz
- renumbered C6 to C10, C7 to C11, C8 to C12, C4 to C2, C9 to C3, C10 to C4, C11 to C5, C12 to C6, C2 to C7, C3 to C8, C5 to C9, JP2 to JP1, JP3 to JP2, JP4 to JP3, JP5 to JP4, JP1 to JP5, R4 to R1, R3 to R2, R5 to R3, U3 to U2, U2 to U3

Commit message: Cleanup and add pin labels AVR
Parts:
- C3, C4: value 22pF -> 20pF
- C5, C6: value 10pF -> 12pF
- Y1: footprint Crystal:Crystal_SMD_MicroCrystal_CC7V-T1A-2Pin_3.2x1.5mm -> Crystal:Crystal_SMD_Abracon_ABM8G-4Pin_3.2x2.5mm
- Y2: footprint Crystal:Crystal_SMD_MicroCrystal_CC7V-T1A-2Pin_3.2x1.5mm -> Crystal:Crystal_Round_D3.0mm_Vertical
Changed lines of the file:
@@
 F 0 "Y1" H 4300 1668 50  0000 C CNN
 F 1 "24MHz" H 4300 1577 50  0000 C CNN
-F 2 "Crystal:Crystal_SMD_MicroCrystal_CC7V-T1A-2Pin_3.2x1.5mm" H 4300 1400 50  0001 C CNN
-F 3 "~" H 4300 1400 50  0001 C CNN
+F 2 "Crystal:Crystal_SMD_Abracon_ABM8G-4Pin_3.2x2.5mm" H 4300 1400 50  0001 C CNN
+F 3 "https://www.mouser.com/datasheet/2/3/C3BQ-2010323.pdf" H 4300 1400 50  0001 C CNN
 	1    4300 1400
 	1    0    0    -1
@@
 P 4500 1650
 F 0 "C4" H 4615 1696 50  0000 L CNN
-F 1 "22pF" H 4615 1605 50  0000 L CNN
+F 1 "20pF" H 4615 1605 50  0000 L CNN
 F 2 "Capacitor_SMD:C_1206_3216Metric" H 4538 1500 50  0001 C CNN
 F 3 "~" H 4500 1650 50  0001 C CNN
@@
 P 4100 1650
 F 0 "C3" H 4215 1696 50  0000 L CNN
-F 1 "22pF" H 4215 1605 50  0000 L CNN
+F 1 "20pF" H 4215 1605 50  0000 L CNN
 F 2 "Capacitor_SMD:C_1206_3216Metric" H 4138 1500 50  0001 C CNN
 F 3 "~" H 4100 1650 50  0001 C CNN
@@
 F 0 "Y2" H 5800 1668 50  0000 C CNN
 F 1 "32768Hz" H 5800 1577 50  0000 C CNN
-F 2 "Crystal:Crystal_SMD_MicroCrystal_CC7V-T1A-2Pin_3.2x1.5mm" H 5800 1400 50  0001 C CNN
-F 3 "~" H 5800 1400 50  0001 C CNN
+F 2 "Crystal:Crystal_Round_D3.0mm_Vertical" H 5800 1400 50  0001 C CNN
+F 3 "https://abracon.com/Resonators/AB38T.pdf" H 5800 1400 50  0001 C CNN
 	1    5800 1400
 	1    0    0    -1
@@
 P 6000 1650
 F 0 "C6" H 6115 1696 50  0000 L CNN
-F 1 "10pF" H 6115 1605 50  0000 L CNN
+F 1 "12pF" H 6115 1605 50  0000 L CNN
 F 2 "Capacitor_SMD:C_1206_3216Metric" H 6038 1500 50  0001 C CNN
 F 3 "~" H 6000 1650 50  0001 C CNN
@@
 P 5600 1650
 F 0 "C5" H 5715 1696 50  0000 L CNN
-F 1 "10pF" H 5715 1605 50  0000 L CNN
+F 1 "12pF" H 5715 1605 50  0000 L CNN
 F 2 "Capacitor_SMD:C_1206_3216Metric" H 5638 1500 50  0001 C CNN
 F 3 "~" H 5600 1650 50  0001 C CNN

Commit message: Update 32768 config and PDF and PNG for AVR
Parts:
- removed C5, C6: 12pF, Capacitor_SMD:C_1206_3216Metric, symbol Device:C
Connections:
- wire segments 49 -> 47
Changed lines of the file:
@@
-	1    0    0    -1
-$EndComp
-$Comp
-L Device:C C4
-U 1 1 61227F49
-P 4500 1650
-F 0 "C4" H 4615 1696 50  0000 L CNN
-F 1 "20pF" H 4615 1605 50  0000 L CNN
-F 2 "Capacitor_SMD:C_1206_3216Metric" H 4538 1500 50  0001 C CNN
-F 3 "~" H 4500 1650 50  0001 C CNN
-	1    4500 1650
-	1    0    0    -1
-$EndComp
-$Comp
-L Device:C C3
-U 1 1 61228826
-P 4100 1650
-F 0 "C3" H 4215 1696 50  0000 L CNN
-F 1 "20pF" H 4215 1605 50  0000 L CNN
-F 2 "Capacitor_SMD:C_1206_3216Metric" H 4138 1500 50  0001 C CNN
-F 3 "~" H 4100 1650 50  0001 C CNN
-	1    4100 1650
 	1    0    0    -1
 $EndComp
 Text Label 4100 950  2    50   ~ 0
 A0
-$Comp
-L power:GND #PWR07
-U 1 1 6122D62F
-P 4100 1800
-F 0 "#PWR07" H 4100 1550 50  0001 C CNN
-F 1 "GND" H 4100 1650 50  0000 C CNN
-F 2 "" H 4100 1800 50  0000 C CNN
-F 3 "" H 4100 1800 50  0000 C CNN
-	1    4100 1800
-	1    0    0    -1
-$EndComp
-$Comp
-L power:GND #PWR08
-U 1 1 6122DCD0
-P 4500 1800
-F 0 "#PWR08" H 4500 1550 50  0001 C CNN
-F 1 "GND" H 4500 1650 50  0000 C CNN
-F 2 "" H 4500 1800 50  0000 C CNN
-F 3 "" H 4500 1800 50  0000 C CNN
-	1    4500 1800
-	1    0    0    -1
-$EndComp
 Text Notes 4600 2150 0    50   ~ 0
 Optional external crystals
-Wire Wire Line
-	4500 1400 4500 1500
 $Comp
 L Jumper:SolderJumper_2_Open JP1
@@
 	1    0    0    -1
 $EndComp
-Connection ~ 4500 1400
 Wire Wire Line
 	4500 950  4500 1150
@@
 Wire Wire Line
 	4150 1400 4100 1400
-Connection ~ 4100 1400
-Wire Wire Line
-	4100 1400 4100 1500
 $Comp
 L Device:Crystal Y2
@@
 	1    0    0    -1
 $EndComp
-$Comp
-L Device:C C6
-U 1 1 6124AFC7
-P 6000 1650
-F 0 "C6" H 6115 1696 50  0000 L CNN
-F 1 "12pF" H 6115 1605 50  0000 L CNN
-F 2 "Capacitor_SMD:C_1206_3216Metric" H 6038 1500 50  0001 C CNN
-F 3 "~" H 6000 1650 50  0001 C CNN
-	1    6000 1650
-	1    0    0    -1
-$EndComp
-$Comp
-L Device:C C5
-U 1 1 6124AFD1
-P 5600 1650
-F 0 "C5" H 5715 1696 50  0000 L CNN
-F 1 "12pF" H 5715 1605 50  0000 L CNN
-F 2 "Capacitor_SMD:C_1206_3216Metric" H 5638 1500 50  0001 C CNN
-F 3 "~" H 5600 1650 50  0001 C CNN
-	1    5600 1650
-	1    0    0    -1
-$EndComp
 Text Label 5600 950  2    50   ~ 0
 F0
-$Comp
-L power:GND #PWR09
-U 1 1 6124AFDC
-P 5600 1800
-F 0 "#PWR09" H 5600 1550 50  0001 C CNN
-F 1 "GND" H 5600 1650 50  0000 C CNN
-F 2 "" H 5600 1800 50  0000 C CNN
-F 3 "" H 5600 1800 50  0000 C CNN
-	1    5600 1800
-	1    0    0    -1
-$EndComp
-$Comp
-L power:GND #PWR010
-U 1 1 6124AFE6
-P 6000 1800
-F 0 "#PWR010" H 6000 1550 50  0001 C CNN
-F 1 "GND" H 6000 1650 50  0000 C CNN
-F 2 "" H 6000 1800 50  0000 C CNN
-F 3 "" H 6000 1800 50  0000 C CNN
-	1    6000 1800
-	1    0    0    -1
-$EndComp
-Wire Wire Line
-	6000 1400 6000 1500
 $Comp
 L Jumper:SolderJumper_2_Open JP3
@@
 	1    0    0    -1
 $EndComp
-Connection ~ 6000 1400
 Wire Wire Line
 	6000 950  6000 1150
@@
 Wire Wire Line
 	5650 1400 5600 1400
-Connection ~ 5600 1400
-Wire Wire Line
-	5600 1400 5600 1500
 Text Label 4800 1150 0    50   ~ 0
 CA1
 Text Label 6300 1150 0    50   ~ 0
 CF1
+Connection ~ 4500 1400
+Wire Wire Line
+	4500 1400 4500 1500
+Connection ~ 4100 1400
+Wire Wire Line
+	4100 1400 4100 1500
+$Comp
+L power:GND #PWR07
+U 1 1 6122D62F
+P 4100 1800
+F 0 "#PWR07" H 4100 1550 50  0001 C CNN
+F 1 "GND" H 4100 1650 50  0000 C CNN
+F 2 "" H 4100 1800 50  0000 C CNN
+F 3 "" H 4100 1800 50  0000 C CNN
+	1    4100 1800
+	1    0    0    -1
+$EndComp
+$Comp
+L power:GND #PWR08
+U 1 1 6122DCD0
+P 4500 1800
+F 0 "#PWR08" H 4500 1550 50  0001 C CNN
+F 1 "GND" H 4500 1650 50  0000 C CNN
+F 2 "" H 4500 1800 50  0000 C CNN
+F 3 "" H 4500 1800 50  0000 C CNN
+	1    4500 1800
+	1    0    0    -1
+$EndComp
+$Comp
+L Device:C C4
+U 1 1 61227F49
+P 4500 1650
+F 0 "C4" H 4615 1696 50  0000 L CNN
+F 1 "20pF" H 4615 1605 50  0000 L CNN
+F 2 "Capacitor_SMD:C_1206_3216Metric" H 4538 1500 50  0001 C CNN
+F 3 "~" H 4500 1650 50  0001 C CNN
+	1    4500 1650
+	1    0    0    -1
+$EndComp
+$Comp
+L Device:C C3
+U 1 1 61228826
+P 4100 1650
+F 0 "C3" H 4215 1696 50  0000 L CNN
+F 1 "20pF" H 4215 1605 50  0000 L CNN
+F 2 "Capacitor_SMD:C_1206_3216Metric" H 4138 1500 50  0001 C CNN
+F 3 "~" H 4100 1650 50  0001 C CNN
+	1    4100 1650
+	1    0    0    -1
+$EndComp
 $EndSCHEMATC
