File: AVR-LORA.sch (KiCad schematic (older format))
At the start: 32 parts, among them J1 Batt, J2 Solar, J3 CONN_01X01, J4 CONN_01X14, J5 CONN_01X14, U1 MCP1700-3302E_SOT23, U2 RFM95HW, U3 AVR128DB28, Y1 24MHz, Y2 32768Hz

Commit message: Update 24MHz crystal config and PDF and PNG for AVR
Parts:
- Y1: symbol Device:Crystal -> Device:Crystal_GND24
Other:
- moved on the sheet: C3, C4
Changed lines of the file:
@@
 I2C pull ups
 $Comp
-L Device:Crystal Y1
+L Device:Crystal_GND24 Y1
 U 1 1 61227560
 P 4300 1400
-F 0 "Y1" H 4300 1668 50  0000 C CNN
-F 1 "24MHz" H 4300 1577 50  0000 C CNN
+F 0 "Y1" H 4300 1800 50  0000 C CNN
+F 1 "24MHz" H 4300 1700 50  0000 C CNN
 F 2 "Crystal:Crystal_SMD_Abracon_ABM8G-4Pin_3.2x2.5mm" H 4300 1400 50  0001 C CNN
 F 3 "https://www.mouser.com/datasheet/2/3/C3BQ-2010323.pdf" H 4300 1400 50  0001 C CNN
@@
 Text Label 4100 950  2    50   ~ 0
 A0
-Text Notes 4600 2150 0    50   ~ 0
+Text Notes 5050 1800 0    50   ~ 0
 Optional external crystals
 $Comp
@@
 Connection ~ 4500 1400
 Wire Wire Line
-	4500 1400 4500 1500
+	4500 1400 4500 1600
 Connection ~ 4100 1400
 Wire Wire Line
-	4100 1400 4100 1500
+	4100 1400 4100 1600
 $Comp
 L power:GND #PWR07
 U 1 1 6122D62F
-P 4100 1800
-F 0 "#PWR07" H 4100 1550 50  0001 C CNN
-F 1 "GND" H 4100 1650 50  0000 C CNN
-F 2 "" H 4100 1800 50  0000 C CNN
-F 3 "" H 4100 1800 50  0000 C CNN
-	1    4100 1800
+P 4100 1900
+F 0 "#PWR07" H 4100 1650 50  0001 C CNN
+F 1 "GND" H 4100 1750 50  0000 C CNN
+F 2 "" H 4100 1900 50  0000 C CNN
+F 3 "" H 4100 1900 50  0000 C CNN
+	1    4100 1900
 	1    0    0    -1
 $EndComp
@@
 L power:GND #PWR08
 U 1 1 6122DCD0
-P 4500 1800
-F 0 "#PWR08" H 4500 1550 50  0001 C CNN
-F 1 "GND" H 4500 1650 50  0000 C CNN
-F 2 "" H 4500 1800 50  0000 C CNN
-F 3 "" H 4500 1800 50  0000 C CNN
-	1    4500 1800
+P 4500 1900
+F 0 "#PWR08" H 4500 1650 50  0001 C CNN
+F 1 "GND" H 4500 1750 50  0000 C CNN
+F 2 "" H 4500 1900 50  0000 C CNN
+F 3 "" H 4500 1900 50  0000 C CNN
+	1    4500 1900
 	1    0    0    -1
 $EndComp
@@
 L Device:C C4
 U 1 1 61227F49
-P 4500 1650
-F 0 "C4" H 4615 1696 50  0000 L CNN
-F 1 "20pF" H 4615 1605 50  0000 L CNN
-F 2 "Capacitor_SMD:C_1206_3216Metric" H 4538 1500 50  0001 C CNN
-F 3 "~" H 4500 1650 50  0001 C CNN
-	1    4500 1650
+P 4500 1750
+F 0 "C4" H 4615 1796 50  0000 L CNN
+F 1 "20pF" H 4615 1705 50  0000 L CNN
+F 2 "Capacitor_SMD:C_1206_3216Metric" H 4538 1600 50  0001 C CNN
+F 3 "~" H 4500 1750 50  0001 C CNN
+	1    4500 1750
 	1    0    0    -1
 $EndComp
@@
 L Device:C C3
 U 1 1 61228826
-P 4100 1650
-F 0 "C3" H 4215 1696 50  0000 L CNN
-F 1 "20pF" H 4215 1605 50  0000 L CNN
-F 2 "Capacitor_SMD:C_1206_3216Metric" H 4138 1500 50  0001 C CNN
-F 3 "~" H 4100 1650 50  0001 C CNN
-	1    4100 1650
+P 4100 1750
+F 0 "C3" H 4215 1796 50  0000 L CNN
+F 1 "20pF" H 4215 1705 50  0000 L CNN
+F 2 "Capacitor_SMD:C_1206_3216Metric" H 4138 1600 50  0001 C CNN
+F 3 "~" H 4100 1750 50  0001 C CNN
+	1    4100 1750
 	1    0    0    -1
 $EndComp

Commit message: Better 24Mhz layout AVR
Parts:
- JP5: value SolderJumper_2_Open -> Close when no MCP1700
Connections:
- wire segments 47 -> 49
Other:
- note added: "C7/C9/C11 are optional"
- note added: "Optional voltage divider\nfor ADC Battery"
- moved on the sheet: C3, C4
Changed lines of the file:
@@
 P 2350 1800
 F 0 "JP5" H 2350 1950 50  0000 C CNN
-F 1 "SolderJumper_2_Open" H 2350 1650 50  0000 C CNN
+F 1 "Close when no MCP1700" H 2350 1650 50  0000 C CNN
 F 2 "Jumper:SolderJumper-2_P1.3mm_Open_Pad1.0x1.5mm" H 2350 1800 50  0001 C CNN
 F 3 "~" H 2350 1800 50  0001 C CNN
@@
 U 1 1 61227560
 P 4300 1400
-F 0 "Y1" H 4300 1800 50  0000 C CNN
-F 1 "24MHz" H 4300 1700 50  0000 C CNN
+F 0 "Y1" H 4300 1950 50  0000 C CNN
+F 1 "24MHz" H 4300 1850 50  0000 C CNN
 F 2 "Crystal:Crystal_SMD_Abracon_ABM8G-4Pin_3.2x2.5mm" H 4300 1400 50  0001 C CNN
 F 3 "https://www.mouser.com/datasheet/2/3/C3BQ-2010323.pdf" H 4300 1400 50  0001 C CNN
@@
 $EndComp
 Text Label 4100 950  2    50   ~ 0
-A0
-Text Notes 5050 1800 0    50   ~ 0
+A1
+Text Notes 5050 1700 0    50   ~ 0
 Optional external crystals
 $Comp
@@
 	4100 950  4100 1150
 Text Label 3800 1150 2    50   ~ 0
-CA0
-Text Label 4500 950  2    50   ~ 0
-A1
+CA1
+Text Label 4500 950  0    50   ~ 0
+A0
 $Comp
 L Jumper:SolderJumper_2_Open JP2
@@
 	5650 1400 5600 1400
 Text Label 4800 1150 0    50   ~ 0
-CA1
+CA0
 Text Label 6300 1150 0    50   ~ 0
 CF1
 Connection ~ 4500 1400
 Wire Wire Line
-	4500 1400 4500 1600
+	4500 1400 4500 1550
 Connection ~ 4100 1400
 Wire Wire Line
-	4100 1400 4100 1600
+	4100 1400 4100 1550
 $Comp
 L power:GND #PWR07
 U 1 1 6122D62F
-P 4100 1900
-F 0 "#PWR07" H 4100 1650 50  0001 C CNN
-F 1 "GND" H 4100 1750 50  0000 C CNN
-F 2 "" H 4100 1900 50  0000 C CNN
-F 3 "" H 4100 1900 50  0000 C CNN
-	1    4100 1900
+P 4100 1850
+F 0 "#PWR07" H 4100 1600 50  0001 C CNN
+F 1 "GND" H 4100 1700 50  0000 C CNN
+F 2 "" H 4100 1850 50  0000 C CNN
+F 3 "" H 4100 1850 50  0000 C CNN
+	1    4100 1850
 	1    0    0    -1
 $EndComp
@@
 L power:GND #PWR08
 U 1 1 6122DCD0
-P 4500 1900
-F 0 "#PWR08" H 4500 1650 50  0001 C CNN
-F 1 "GND" H 4500 1750 50  0000 C CNN
-F 2 "" H 4500 1900 50  0000 C CNN
-F 3 "" H 4500 1900 50  0000 C CNN
-	1    4500 1900
+P 4500 1850
+F 0 "#PWR08" H 4500 1600 50  0001 C CNN
+F 1 "GND" H 4500 1700 50  0000 C CNN
+F 2 "" H 4500 1850 50  0000 C CNN
+F 3 "" H 4500 1850 50  0000 C CNN
+	1    4500 1850
 	1    0    0    -1
 $EndComp
@@
 L Device:C C4
 U 1 1 61227F49
-P 4500 1750
-F 0 "C4" H 4615 1796 50  0000 L CNN
-F 1 "20pF" H 4615 1705 50  0000 L CNN
-F 2 "Capacitor_SMD:C_1206_3216Metric" H 4538 1600 50  0001 C CNN
-F 3 "~" H 4500 1750 50  0001 C CNN
-	1    4500 1750
-	1    0    0    -1
+P 4500 1700
+F 0 "C4" H 4615 1746 50  0000 L CNN
+F 1 "20pF" H 4615 1655 50  0000 L CNN
+F 2 "Capacitor_SMD:C_1206_3216Metric" H 4538 1550 50  0001 C CNN
+F 3 "~" H 4500 1700 50  0001 C CNN
+	1    4500 1700
+	1    0    0    -1
+$EndComp
+$Comp
+L power:GND #PWR?
+U 1 1 6134A299
+P 4300 1600
+F 0 "#PWR?" H 4300 1350 50  0001 C CNN
+F 1 "GND" H 4300 1450 50  0000 C CNN
+F 2 "" H 4300 1600 50  0000 C CNN
+F 3 "" H 4300 1600 50  0000 C CNN
+	1    4300 1600
+	1    0    0    -1
+$EndComp
+$Comp
+L power:GND #PWR?
+U 1 1 6134B029
+P 4300 1200
+F 0 "#PWR?" H 4300 950 50  0001 C CNN
+F 1 "GND" H 4300 1050 50  0000 C CNN
+F 2 "" H 4300 1200 50  0000 C CNN
+F 3 "" H 4300 1200 50  0000 C CNN
+	1    4300 1200
+	-1   0    0    1
 $EndComp
 $Comp
 L Device:C C3
 U 1 1 61228826
-P 4100 1750
-F 0 "C3" H 4215 1796 50  0000 L CNN
-F 1 "20pF" H 4215 1705 50  0000 L CNN
-F 2 "Capacitor_SMD:C_1206_3216Metric" H 4138 1600 50  0001 C CNN
-F 3 "~" H 4100 1750 50  0001 C CNN
-	1    4100 1750
-	1    0    0    -1
-$EndComp
+P 4100 1700
+F 0 "C3" H 3850 1750 50  0000 L CNN
+F 1 "20pF" H 3800 1650 50  0000 L CNN
+F 2 "Capacitor_SMD:C_1206_3216Metric" H 4138 1550 50  0001 C CNN
+F 3 "~" H 4100 1700 50  0001 C CNN
+	1    4100 1700
+	1    0    0    -1
+$EndComp
+Connection ~ 4100 1550
+Wire Wire Line
+	4100 1550 4100 1750
+Connection ~ 4500 1550
+Wire Wire Line
+	4500 1550 4500 1750
+Text Notes 8350 3350 0    50   ~ 0
+Optional voltage divider\nfor ADC Battery
+Text Notes 1100 2550 0    50   ~ 0
+C7/C9/C11 are optional
 $EndSCHEMATC
