File: AVR-LORA.sch (KiCad schematic (older format))
At the start: 32 parts, among them J1 Batt, J2 Solar, J3 CONN_01X01, J4 CONN_01X14, J5 CONN_01X14, U1 MCP1700-3302E_SOT23, U2 RFM95HW, U3 AVR128DB28, Y1 24MHz, Y2 32768Hz

Commit message: Add SMA connector
Parts:
- J3: value CONN_01X01 -> SMA; footprint Connector_PinHeader_2.54mm:PinHeader_1x01_P2.54mm_Vertical -> Connector_Coaxial:SMA_Amphenol_132134_Vertical
Changed lines of the file:
@@
 P 4700 2950
 F 0 "J3" H 4700 3050 50  0000 C CNN
-F 1 "CONN_01X01" V 4800 2950 50  0000 C CNN
-F 2 "Connector_PinHeader_2.54mm:PinHeader_1x01_P2.54mm_Vertical" H 4700 2950 50  0001 C CNN
+F 1 "SMA" V 4800 2950 50  0000 C CNN
+F 2 "Connector_Coaxial:SMA_Amphenol_132134_Vertical" H 4700 2950 50  0001 C CNN
 F 3 "" H 4700 2950 50  0001 C CNN
 	1    4700 2950
@@
 $EndComp
 $Comp
-L power:GND #PWR?
+L power:GND #PWR0101
 U 1 1 6134A299
 P 4300 1600
-F 0 "#PWR?" H 4300 1350 50  0001 C CNN
+F 0 "#PWR0101" H 4300 1350 50  0001 C CNN
 F 1 "GND" H 4300 1450 50  0000 C CNN
 F 2 "" H 4300 1600 50  0000 C CNN
@@
 $EndComp
 $Comp
-L power:GND #PWR?
+L power:GND #PWR0102
 U 1 1 6134B029
 P 4300 1200
-F 0 "#PWR?" H 4300 950 50  0001 C CNN
+F 0 "#PWR0102" H 4300 950 50  0001 C CNN
 F 1 "GND" H 4300 1050 50  0000 C CNN
 F 2 "" H 4300 1200 50  0000 C CNN

Commit message: GND SMA connector in schema
Parts:
- J3: symbol STM-LORA-rescue:CONN_01X01 -> Connector:Conn_Coaxial
Changed lines of the file:
@@
 	8000 2150 8000 1850
 $Comp
-L STM-LORA-rescue:CONN_01X01 J3
+L Connector:Conn_Coaxial J3
 U 1 1 593BCF25
 P 4700 2950
@@
 Text Notes 1100 2550 0    50   ~ 0
 C7/C9/C11 are optional
+$Comp
+L power:GND #PWR?
+U 1 1 61256928
+P 4900 2950
+F 0 "#PWR?" H 4900 2700 50  0001 C CNN
+F 1 "GND" H 4900 2800 50  0000 C CNN
+F 2 "" H 4900 2950 50  0000 C CNN
+F 3 "" H 4900 2950 50  0000 C CNN
+	1    4900 2950
+	0    -1   -1   0
+$EndComp
 $EndSCHEMATC

Commit message: Add capacitors to 32768 crystal for 0805 version
Parts:
- added C5, C6: 10pF, Capacitor_SMD:C_1206_3216Metric, symbol Device:C
Changed lines of the file:
@@
 Sheet 1 1
 Title "AVR RFM95 Board"
-Date "2021-08-17"
-Rev "1.0"
+Date "2021-09-19"
+Rev "1.1"
 Comp "http://v7f.eu"
 Comment1 ""
@@
 Text Label 4100 950  2    50   ~ 0
 A1
-Text Notes 5050 1700 0    50   ~ 0
+Text Notes 4600 700  0    50   ~ 0
 Optional external crystals
 $Comp
@@
 C7/C9/C11 are optional
 $Comp
-L power:GND #PWR?
+L power:GND #PWR09
 U 1 1 61256928
 P 4900 2950
-F 0 "#PWR?" H 4900 2700 50  0001 C CNN
+F 0 "#PWR09" H 4900 2700 50  0001 C CNN
 F 1 "GND" H 4900 2800 50  0000 C CNN
 F 2 "" H 4900 2950 50  0000 C CNN
@@
 	0    -1   -1   0
 $EndComp
+$Comp
+L Device:C C6
+U 1 1 6147B2E9
+P 6000 1550
+F 0 "C6" H 6115 1596 50  0000 L CNN
+F 1 "10pF" H 6115 1505 50  0000 L CNN
+F 2 "Capacitor_SMD:C_1206_3216Metric" H 6038 1400 50  0001 C CNN
+F 3 "~" H 6000 1550 50  0001 C CNN
+	1    6000 1550
+	1    0    0    -1
+$EndComp
+Connection ~ 6000 1400
+$Comp
+L Device:C C5
+U 1 1 6147C02E
+P 5600 1550
+F 0 "C5" H 5350 1600 50  0000 L CNN
+F 1 "10pF" H 5300 1500 50  0000 L CNN
+F 2 "Capacitor_SMD:C_1206_3216Metric" H 5638 1400 50  0001 C CNN
+F 3 "~" H 5600 1550 50  0001 C CNN
+	1    5600 1550
+	1    0    0    -1
+$EndComp
+Connection ~ 5600 1400
+$Comp
+L power:GND #PWR0103
+U 1 1 6147EC70
+P 5600 1700
+F 0 "#PWR0103" H 5600 1450 50  0001 C CNN
+F 1 "GND" H 5600 1550 50  0000 C CNN
+F 2 "" H 5600 1700 50  0000 C CNN
+F 3 "" H 5600 1700 50  0000 C CNN
+	1    5600 1700
+	1    0    0    -1
+$EndComp
+$Comp
+L power:GND #PWR0104
+U 1 1 614806B9
+P 6000 1700
+F 0 "#PWR0104" H 6000 1450 50  0001 C CNN
+F 1 "GND" H 6000 1550 50  0000 C CNN
+F 2 "" H 6000 1700 50  0000 C CNN
+F 3 "" H 6000 1700 50  0000 C CNN
+	1    6000 1700
+	1    0    0    -1
+$EndComp
 $EndSCHEMATC
