File: AVR-LORA-805.kicad_pcb (KiCad board)
At the start: 2 copper layers, 51.7 x 29.2 mm, 36 parts, among them J1 Batt, J2 Solar, J3 SMA, J4 CONN_01X14, J5 CONN_01X14, U1 MCP1700-3302E_SOT23, U2 RFM95HW, U3 AVR128DB28, Y1 24MHz, Y2 32768Hz

Commit message: Improve silk 805
Routing:
- net GND: track 72.3 -> 68.5 mm, vias 42 -> 47
- net /3V3: track 102.2 -> 100.8 mm
- net /D5: track 37.9 -> 39.0 mm
- net /C3: track 38.2 -> 39.1 mm
- net /A3: track 30.2 -> 31.1 mm
- net /A1: track 15.2 -> 16.0 mm
- net /D2: track 28.0 -> 27.3 mm
