File: AVR-LORA.kicad_sch (KiCad schematic)
At the start: 34 parts, among them J1 Batt, J2 Solar, J3 SMA, J4 CONN_01X14, J5 CONN_01X14, U1 MCP1700-3302E_SOT23, U2 RFM95HW, U3 AVR128DB28, Y1 24MHz, Y2 32768Hz

Commit message: Minor cleanups AVR 805 version
Connections:
- no-connect marks 3 -> 4
Changed lines of the file:
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@@
 		(at 147.32 96.52)
+	)
+	(no_connect
+		(at 198.12 34.29)
 	)
 	(wire
@@
 					(size 1.524 1.524)
 				)
-			)
-		)
+				(hide yes)
+			)
+		)
